Commit message: changed to MPPI , no tank turns, Dubin, reliable navigation with faster speeds

File: src/argo_mini/urdf/argo_mini.urdf (robot description, URDF)
Before this commit: robot robot_chassis, 18 links, 17 joints
Links:
- link left_wheel_link: geometry collision cylinder length=0.05 radius=0.0762; visual cylinder length=0.05 radius=0.0762
- link right_wheel_link: geometry collision cylinder length=0.05 radius=0.0762; visual cylinder length=0.05 radius=0.0762

Commit message: Working prototype 100 percent

File: src/argo_mini/urdf/argo_mini.urdf (robot description, URDF)
Before this commit: robot robot_chassis, 18 links, 17 joints
Joints:
- joint lidar_joint: origin xyz=0.1375 0 0.1095 rpy=0 0 3.141592653589793 -> xyz=0.085 0 0.12 rpy=0 0 0
