Commit message: Replace URDF with xacro-based model; update frame names throughout
- Add argo_mini.xacro with full chassis model (plates, standoffs, wheels,
  casters, lidar, depth camera) including Gazebo plugins
- Regenerate argo_mini.urdf from xacro (659 lines → 659 lines, all macros expanded)
- Frame renames: laser→lidar_link, camera_depth_optical_frame→depth_camera_optical_frame
- serial_bridge: publish odom→base_footprint (was base_link); robot_state_publisher
  now handles base_footprint→base_link via URDF fixed joint
- start_slam.sh: replace static TF publisher with robot_state_publisher.launch.py;
  rplidar frame_id laser→lidar_link
- start_argo_nav.sh: rplidar frame_id laser→lidar_link; camera TF bridge frame
  camera_depth_optical_frame→depth_camera_optical_frame; move camera TF bridge
  before camera launch so depth_safety_shield TF lookups never fail

Co-Authored-By: Claude Sonnet 4.6 <noreply@anthropic.com>

File: src/argo_mini/urdf/argo_mini.urdf (robot description, URDF)
Before this commit: robot argo_mini, 6 links, 5 joints
Links:
- removed link camera_depth_optical_frame
- removed link laser
- removed link left_wheel
- removed link right_wheel
- added link base_footprint
- added link caster_mount_rl_link, mass 0.02; collision cylinder length=0.005 radius=0.018; visual cylinder length=0.005 radius=0.018
- added link caster_mount_rr_link, mass 0.02; collision cylinder length=0.005 radius=0.018; visual cylinder length=0.005 radius=0.018
- added link caster_wheel_rl_link, mass 0.08; collision cylinder length=0.02 radius=0.03; visual cylinder length=0.02 radius=0.03
- added link caster_wheel_rr_link, mass 0.08; collision cylinder length=0.02 radius=0.03; visual cylinder length=0.02 radius=0.03
- added link caster_yaw_rl_link, mass 0.03; collision box size=0.022 0.012 0.025; visual box size=0.022 0.012 0.025
- added link caster_yaw_rr_link, mass 0.03; collision box size=0.022 0.012 0.025; visual box size=0.022 0.012 0.025
- added link depth_camera_optical_frame
- added link left_wheel_link, mass 1.5; collision cylinder length=0.05 radius=0.085; visual cylinder length=0.05 radius=0.085
- added link lidar_link, mass 0.19; collision cylinder length=0.041 radius=0.038; visual cylinder length=0.041 radius=0.038
- added link right_wheel_link, mass 1.5; collision cylinder length=0.05 radius=0.085; visual cylinder length=0.05 radius=0.085
- added link standoff_fl_link, mass 0.05; collision box size=0.025 0.025 0.16; visual box size=0.025 0.025 0.16
- added link standoff_fr_link, mass 0.05; collision box size=0.025 0.025 0.16; visual box size=0.025 0.025 0.16
- added link standoff_rl_link, mass 0.05; collision box size=0.025 0.025 0.16; visual box size=0.025 0.025 0.16
- added link standoff_rr_link, mass 0.05; collision box size=0.025 0.025 0.16; visual box size=0.025 0.025 0.16
- added link upper_plate_link, mass 2.0; collision box size=0.03749999999999998 0.16749999999999998 0.003; collision box size=0.03749999999999998 0.16749999999999998 0.003
- link base_link: mass 12.0 -> 2.0; geometry collision box size=0.10999999999999999 0.435 0.003; collision box size=0.19 0.34500000000000003 0.003
- link camera_link: mass 0.10 -> 0.1; geometry collision box size=0.025 0.09 0.025; visual box size=0.025 0.09 0.025
Joints:
- removed joint camera_depth_optical_joint
- removed joint laser_joint
- added joint base_footprint_to_base_link: type fixed, parent base_footprint, child base_link, origin xyz=0 0 0.06 rpy=0 0 0
- added joint camera_optical_joint: type fixed, parent camera_link, child depth_camera_optical_frame, origin xyz=0 0 0 rpy=-1.5707963267948966 0 -1.5707963267948966
- added joint caster_mount_rl_joint: type fixed, parent base_link, child caster_mount_rl_link, origin xyz=-0.16 0.135 0 rpy=0 0 0
- added joint caster_mount_rr_joint: type fixed, parent base_link, child caster_mount_rr_link, origin xyz=-0.16 -0.135 0 rpy=0 0 0
- added joint caster_wheel_rl_joint: type continuous, parent caster_yaw_rl_link, child caster_wheel_rl_link, origin xyz=-0.012 0 -0.025 rpy=0 0 0, axis 0 1 0
- added joint caster_wheel_rr_joint: type continuous, parent caster_yaw_rr_link, child caster_wheel_rr_link, origin xyz=-0.012 0 -0.025 rpy=0 0 0, axis 0 1 0
- added joint caster_yaw_rl_joint: type continuous, parent caster_mount_rl_link, child caster_yaw_rl_link, origin xyz=0 0 -0.005 rpy=0 0 0, axis 0 0 1
- added joint caster_yaw_rr_joint: type continuous, parent caster_mount_rr_link, child caster_yaw_rr_link, origin xyz=0 0 -0.005 rpy=0 0 0, axis 0 0 1
- added joint lidar_joint: type fixed, parent base_link, child lidar_link, origin xyz=0.1375 0 0.1095 rpy=0 0 0
- added joint lower_plate_to_upper_plate: type fixed, parent base_link, child upper_plate_link, origin xyz=0 0 0.11 rpy=0 0 0
- added joint standoff_fl_joint: type fixed, parent base_link, child standoff_fl_link, origin xyz=0.22 0.1925 0.003 rpy=0 0 0
- added joint standoff_fr_joint: type fixed, parent base_link, child standoff_fr_link, origin xyz=0.22 -0.1925 0.003 rpy=0 0 0
- added joint standoff_rl_joint: type fixed, parent base_link, child standoff_rl_link, origin xyz=-0.07999999999999999 0.135 0.003 rpy=0 0 0
- added joint standoff_rr_joint: type fixed, parent base_link, child standoff_rr_link, origin xyz=-0.07999999999999999 -0.135 0.003 rpy=0 0 0
- joint camera_joint: origin xyz=0.22 0.0 0.15 rpy=0.0 0.0 0.0 -> xyz=0.2575 0 0.170 rpy=0 0 0
- joint left_wheel_joint: axis 0 0 1 -> 0 1 0; child left_wheel -> left_wheel_link; limit (none) -> effort=10.0 velocity=10.0; origin xyz=0.0 0.225 0.0 rpy=-1.5708 0.0 0.0 -> xyz=0.05500000000000002 0.1975 0.02500000000000001 rpy=0 0 0
- joint right_wheel_joint: axis 0 0 1 -> 0 1 0; child right_wheel -> right_wheel_link; limit (none) -> effort=10.0 velocity=10.0; origin xyz=0.0 -0.225 0.0 rpy=-1.5708 0.0 0.0 -> xyz=0.05500000000000002 -0.1975 0.02500000000000001 rpy=0 0 0

Commit message: Restore lidar yaw=π (connector faces rear)
Co-Authored-By: Claude Sonnet 4.6 <noreply@anthropic.com>

File: src/argo_mini/urdf/argo_mini.urdf (robot description, URDF)
Before this commit: robot robot_chassis, 18 links, 17 joints
Joints:
- joint lidar_joint: origin xyz=0.1375 0 0.1095 rpy=0 0 0 -> xyz=0.1375 0 0.1095 rpy=0 0 3.141592653589793

Commit message: Add ceiling localization: detector, mount calibration, map builder
In a restaurant everything at lidar height moves -- chairs, bags, people,
nudged tables -- so the laser map is built on furniture that relocates
hourly. The ceiling is the only rigid structure in the building. This runs
alongside the RPLidar + slam_toolbox stack rather than replacing it, and
will publish a standard map->odom correction so Nav2 works unchanged.

Three nodes:
  ceiling_features     lights from RGB, ceiling plane from depth
  ceiling_calibrate    mount tilt and lean, from one view of the plane
  ceiling_map_builder  mount azimuth as a 2D hand-eye solve, plus the map

Depth for the plane, RGB for the landmarks: a fixture is flat against the
ceiling and a 25 mm pipe at 3.6 m is inside the noise, so neither shows up
as usable geometry in depth -- and depth is capped at 4.095 m, which the
tilted far half of the frame exceeds anyway.

The camera is mounted ~24 deg off vertical, fixed in hardware. The static
TF said roll=0 pitch=0 yaw=0 in all nine launch paths and the URDF carried
a forward-facing optical rpy; both now carry the measured mount rotation.

First live run of the detector (see CEILING_LOCALIZATION.md):

  - fit_plane cost 1680 ms and ran on every depth frame at 10.6 Hz, on the
    same single-threaded executor as the landmark path. The node published
    1.4 Hz while the camera offered 6.3 Hz of RGB. Every hypothesis is
    scored the same way against the same points, so the 120 RANSAC
    hypotheses collapse into one (points x hypotheses) product -- ~16x
    faster -- and the fit is now throttled to plane_rate_hz, which costs
    nothing because the mount is rigid and the plane is smoothed anyway.

  - Refitting on the inliers with a shrinking band made it more accurate as
    well as faster: the coarse fit was biasing the plane itself, reading
    tilt 25.7 deg where the refined fit gives 23.2 deg against 23.8 deg
    measured by hand. Landmark jitter went 6.0 mm -> 1.8 mm, output 4.2 Hz.

  - ceiling_calibrate carried its own copy of the same slow estimator and
    now delegates. That node converts the ceiling normal into the mount TF,
    so two nodes fitting one ceiling by different methods is exactly how
    the TF and the landmark projection drift apart.

Still open: the azimuth has not been checked against the installed
+92.361 deg, which needs a drive rather than a bench check, and the
localizer that publishes map->odom is not started.

Co-Authored-By: Claude Opus 5 <noreply@anthropic.com>

File: src/argo_mini/urdf/argo_mini.urdf (robot description, URDF)
Before this commit: robot robot_chassis, 18 links, 17 joints
Joints:
- joint camera_optical_joint: origin xyz=0 0 0 rpy=-1.5707963267948966 0 -1.5707963267948966 -> xyz=0 0 0 rpy=0.417281 -0.018276 1.611996

File: src/argo_mini/urdf/argo_mini.xacro (robot description, xacro)
@@ -288,5 +288,8 @@
     <parent link="camera_link"/>
     <child link="depth_camera_optical_frame"/>
-    <origin xyz="0 0 0" rpy="${-pi/2} 0 ${-pi/2}"/>
+    <!-- HP60C faces UP, tilted 23.9 deg off vertical (fixed in hardware).
+         Measured from the ceiling plane by `ros2 run argo_mini ceiling_calibrate`;
+         was the forward-facing optical rpy, which did not match the mount. -->
+    <origin xyz="0 0 0" rpy="0.417281 -0.018276 1.611996"/>
   </joint>
   <gazebo reference="base_link"><material>Gazebo/Grey</material></gazebo>
