Commit message: xarco change.

File: src/argo_mini/urdf/argo_mini.xacro (robot description, xacro)
@@ -261,5 +261,5 @@
     <parent link="base_link"/>
     <child  link="lidar_link"/>
-    <origin xyz="${lidar_x} 0 ${lidar_max_top_above_lower_chassis - lidar_height/2.0}" rpy="0 0 ${pi}"/>
+    <origin xyz="${lidar_x} 0 ${lidar_max_top_above_lower_chassis - lidar_height/2.0}" rpy="0 0 0"/>
   </joint>
   <link name="camera_link">

Commit message: revert lidar position.

File: src/argo_mini/urdf/argo_mini.xacro (robot description, xacro)
@@ -261,5 +261,5 @@
     <parent link="base_link"/>
     <child  link="lidar_link"/>
-    <origin xyz="${lidar_x} 0 ${lidar_max_top_above_lower_chassis - lidar_height/2.0}" rpy="0 0 0"/>
+    <origin xyz="${lidar_x} 0 ${lidar_max_top_above_lower_chassis - lidar_height/2.0}" rpy="0 0 ${pi}"/>
   </joint>
   <link name="camera_link">
